File: schema.sch (EAGLE design)
At the start: 8 parts, among them IC1 RT9011-CMGJ6, U1 ESP-32S, X1 FH12-24S-0.5SH, X2 C-GRID-02-70543

Commit message: parts update
Parts:
- removed X1: FH12-24S-0.5SH, con-hirose:FH12-24S-0.5SH
- added C4: 0.1uF, rcl:C-EUC0805
- added J1: FH12-24S-0.5SH(55), water-lib:FH12-24S-0.5SH(55)
- added R2: 10k, rcl:R-EU_R0805
- added S1: (no value), switch-omron:10-XX
- added S2: (no value), switch:255SB
- IC1: device RT9011-CMGJ6:RT9011-CMGJ6 -> water-lib:RT9011-CMGJ6
- R1: value (none) -> 1k
- U1: device esp32s:ESP-32S -> water-lib:ESP-32S
Connections:
- new net EN: C4.1, R2.1, S1.S, S1.S1, U1.EN
- new net N$2: U1.GND@4
- new net N$3: S2.P, X2-2.S
- net +3V3: now also R2.2, S2.S; no longer X2-2.S
- net GND: now also C4.2, S1.P, S1.P1; no longer U1.GND@4

Commit message: 5v dc/dc
Parts:
- added C5, C6: 22uF, rcl:C-EUC0805
- added D1: BAT60J, diode:BAT60J
- added IC2: SX1308, water-lib:SX1308
- added L1: 22uH, rcl:L-EU0204/5
- added R3: 10k, rcl:R-EU_R0805
- added R4: 1363, rcl:R-EU_R0805
Connections:
- new net +5V: C6.1, D1.A, R3.2
- new net N$4: D1.C, IC2.SW, L1.1
- new net N$5: IC2.FB, R3.1, R4.2
- net +3V3: now also C5.2, IC2.EN, IC2.IN, L1.2
- net CAM_PWR: now also U1.IO35
- net GND: now also C5.1, C6.2, IC2.GND, R4.1
Other:
- moved on the sheet: J1

Commit message: Added new components
Parts:
- added J2: C10418, water-lib:C10418
- added U2: CH340ESMD, water-lib:CH340ESMD
Connections:
- new net D+: J2.D+, U2.UD+
- new net D-: J2.D-, U2.UD-
- new net N$10: J2.ID
- new net N$11: J2.MH1, J2.MH2, J2.MH3, J2.MH4
- net +5V: now also J2.VBUS
- net GND: now also J2.GND, U2.GND
Changed lines of the file:
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@@
 <?xml version="1.0" encoding="utf-8"?>
 <!DOCTYPE eagle SYSTEM "eagle.dtd">
-<eagle version="9.4.2">
+<eagle version="9.5.0">
 <drawing>
 <settings>
@@
 <part name="GND10" library="supply1" library_urn="urn:adsk.eagle:library:371" deviceset="GND" device=""/>
 <part name="C6" library="rcl" library_urn="urn:adsk.eagle:library:334" deviceset="C-EU" device="C0805" package3d_urn="urn:adsk.eagle:package:23617/2" value="22uF"/>
+<part name="U2" library="water-lib" deviceset="CH340E" device="SMD" package3d_urn="urn:adsk.eagle:package:3661278/1"/>
+<part name="J2" library="water-lib" deviceset="C10418" device=""/>
 </parts>
 <sheets>
@@
 <attribute name="NAME" x="49.784" y="180.721" size="1.778" layer="95"/>
 <attribute name="VALUE" x="49.784" y="175.641" size="1.778" layer="96"/>
+</instance>
+<instance part="U2" gate="G$1" x="-22.86" y="40.64" smashed="yes">
+<attribute name="NAME" x="-26.67" y="25.4" size="1.778" layer="95"/>
+</instance>
+<instance part="J2" gate="G$1" x="-76.2" y="60.96" smashed="yes" rot="R270">
+<attribute name="NAME" x="-68.58" y="39.37" size="1.778" layer="95" rot="R270" align="center-left"/>
+<attribute name="VALUE" x="-71.12" y="39.37" size="1.778" layer="96" rot="R270" align="center-left"/>
 </instance>
 </instances>
@@
 <junction x="55.88" y="162.56"/>
 </segment>
+<segment>
+<pinref part="U2" gate="G$1" pin="GND"/>
+<wire x1="-36.83" y1="40.64" x2="-43.18" y2="40.64" width="0.1524" layer="91"/>
+<label x="-43.18" y="40.64" size="1.778" layer="95"/>
+</segment>
+<segment>
+<pinref part="J2" gate="G$1" pin="GND"/>
+<wire x1="-81.28" y1="60.96" x2="-81.28" y2="63.5" width="0.1524" layer="91"/>
+<label x="-81.28" y="63.5" size="1.778" layer="95" rot="R90"/>
+</segment>
 </net>
 <net name="N$1" class="0">
@@
 <label x="43.18" y="193.04" size="1.778" layer="95" rot="R180" xref="yes"/>
 </segment>
-</net>
+<segment>
+<pinref part="J2" gate="G$1" pin="VBUS"/>
+<wire x1="-76.2" y1="60.96" x2="-76.2" y2="63.5" width="0.1524" layer="91"/>
+<label x="-76.2" y="63.5" size="1.778" layer="95" rot="R90"/>
+</segment>
+</net>
+<net name="D+" class="0">
+<segment>
+<pinref part="U2" gate="G$1" pin="UD+"/>
+<wire x1="-36.83" y1="50.8" x2="-68.58" y2="50.8" width="0.1524" layer="91"/>
+<wire x1="-68.58" y1="50.8" x2="-68.58" y2="71.12" width="0.1524" layer="91"/>
+<wire x1="-68.58" y1="71.12" x2="-78.74" y2="71.12" width="0.1524" layer="91"/>
+<pinref part="J2" gate="G$1" pin="D+"/>
+<wire x1="-78.74" y1="71.12" x2="-78.74" y2="60.96" width="0.1524" layer="91"/>
+</segment>
+</net>
+<net name="D-" class="0">
+<segment>
+<pinref part="U2" gate="G$1" pin="UD-"/>
+<wire x1="-36.83" y1="45.72" x2="-68.58" y2="45.72" width="0.1524" layer="91"/>
+<wire x1="-68.58" y1="45.72" x2="-68.58" y2="25.4" width="0.1524" layer="91"/>
+<wire x1="-68.58" y1="25.4" x2="-76.2" y2="25.4" width="0.1524" layer="91"/>
+<pinref part="J2" gate="G$1" pin="D-"/>
+<wire x1="-76.2" y1="25.4" x2="-76.2" y2="35.56" width="0.1524" layer="91"/>
+</segment>
+</net>
+<net name="N$10" class="0">
+<segment>
+<pinref part="J2" gate="G$1" pin="ID"/>
+<wire x1="-78.74" y1="35.56" x2="-78.74" y2="33.02" width="0.1524" layer="91"/>
+</segment>
+</net>
+<net name="N$11" class="0">
+<segment>
+<pinref part="J2" gate="G$1" pin="MH1"/>
+<pinref part="J2" gate="G$1" pin="MH3"/>
+<wire x1="-81.28" y1="35.56" x2="-83.82" y2="35.56" width="0.1524" layer="91"/>
+<wire x1="-83.82" y1="35.56" x2="-93.98" y2="35.56" width="0.1524" layer="91"/>
+<junction x="-83.82" y="35.56"/>
+<pinref part="J2" gate="G$1" pin="MH4"/>
+<wire x1="-93.98" y1="35.56" x2="-93.98" y2="60.96" width="0.1524" layer="91"/>
+<wire x1="-93.98" y1="60.96" x2="-86.36" y2="60.96" width="0.1524" layer="91"/>
+<pinref part="J2" gate="G$1" pin="MH2"/>
+<wire x1="-86.36" y1="60.96" x2="-83.82" y2="60.96" width="0.1524" layer="91"/>
+<junction x="-86.36" y="60.96"/>
+</segment>
+</net>

Commit message: Added USB-Serial to main design
Parts:
- removed C1, C2, C3: 0.1uF, rcl:C-EUC0805
- removed C5, C6: 22uF, rcl:C-EUC0805
- removed D1: BAT60J, diode:BAT60J
- removed IC1: RT9011-CMGJ6, water-lib:RT9011-CMGJ6
- removed IC2: SX1308, water-lib:SX1308
- removed J2: C10418, water-lib:C10418
- removed L1: 22uH, rcl:L-EU0204/5
- removed R1: 1k, rcl:R-EU_R0805
- removed R3: 10k, rcl:R-EU_R0805
- removed R4: 1363, rcl:R-EU_R0805
- removed S2: (no value), switch:255SB
- removed U2: CH340ESMD, water-lib:CH340ESMD
- removed X2: C-GRID-02-70543, con-molex:C-GRID-02-70543
- added C10, C9: .1uF, rcl:C-EUC0805
- added C7, C8: 10uF, rcl:C-EUC0805
- added F1: SMD0805-020-16V, water-lib:SMD0805-020-16V
- added IC3: HT7333, water-lib:HT7333
- added J3: C10418, water-lib:C10418
- added LED1, LED2, LED3, LED4: (no value), led:LEDCHIP-LED0805
- added R5: 2k, rcl:R-EU_R0805
- added R6, R7, R8: 1K5, rcl:R-EU_R0805
- added U3: CH340ESMD, water-lib:CH340ESMD
Connections:
- removed net +1V2: C2.2, IC1.VOUT2
- removed net +2V8: C3.2, IC1.VOUT1
- removed net +5V: C6.1, D1.A, J2.VBUS, R3.2
- removed net CAM_PWR: R1.1, U1.IO35
- removed net D+: J2.D+, U2.UD+
- removed net D-: J2.D-, U2.UD-
- removed net N$1: IC1.EN1, IC1.EN2, R1.2
- removed net N$10: J2.ID
- removed net N$11: J2.MH1, J2.MH2, J2.MH3, J2.MH4
- removed net N$2: U1.GND@4
- removed net N$3: S2.P, X2-2.S
- removed net N$4: D1.C, IC2.SW, L1.1
- removed net N$5: IC2.FB, R3.1, R4.2
- new net +5V1: C7.1, F1.2, IC3.IN, LED1.A
- new net 3V3: C10.1, C8.1, C9.2, IC3.OUT, LED3.A, LED4.A, U3.V3, U3.VCC
- new net 5V-USB: F1.1, J3.VBUS
- new net CTS: U3.CTS
- new net D+1: J3.D+, U3.UD+
- new net D-1: J3.D-, U3.UD-
- new net MH: J3.MH1, J3.MH2, J3.MH3, J3.MH4
- new net N$12: LED3.C, R7.2
- new net N$13: LED4.C, R8.1
- new net N$7: LED1.C, R5.2
- new net N$8: R6.1, U3.TNOW
- new net N$9: LED2.A, R6.2
- new net NC1: J3.ID
- new net RTS: U3.RTS
- new net RX: R7.1, U1.U0TXD, U3.RX
- new net TX: R8.2, U1.U0RXD, U3.TX
- net +3V3: no longer C1.1, C5.2, IC1.VIN, IC2.EN, IC2.IN, L1.2, S2.S
- net GND: now also C10.2, C7.2, C8.2, C9.1, IC3.GND, J3.GND, LED2.C, R5.1, U1.GND@4, U3.GND; no longer C1.2, C2.1, C3.1, C5.1, C6.2, IC2.GND, J2.GND, R4.1, U2.GND, X2-1.S
Other:
- moved on the sheet: C4, J1, R2, S1

Commit message: Added PSRAM
Parts:
- added C1: 0.1uF, rcl:C-EUC0805
- added IC1: IPS6404L-SQ-SPN, water-lib:IPS6404L-SQ-SPN
- added R1: 10k, rcl:R-EU_R0805
Connections:
- new net IO16: IC1.#CE, R1.1, U1.IO16
- new net PSRAM_CLK: IC1.SCLK, U1.IO17
- new net SD0: IC1.SO/SIO[1], U1.SD0
- new net SD1: IC1.SI/SIO[0], U1.SD1
- new net SD2: IC1.SIO[3], U1.SD2
- new net SD3: IC1.SIO[2], U1.SD3
- net +3V3: now also C1.1, IC1.VDD, R1.2
- net GND: now also C1.2, IC1.VSS
Changed lines of the file:
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@@
 <part name="+3V3" library="supply1" library_urn="urn:adsk.eagle:library:371" deviceset="+3V3" device=""/>
 <part name="GND4" library="supply1" library_urn="urn:adsk.eagle:library:371" deviceset="GND" device=""/>
-<part name="GND5" library="supply1" library_urn="urn:adsk.eagle:library:371" deviceset="GND" device=""/>
+<part name="GND5" library="supply1" library_urn="urn:adsk.eagle:library:371" deviceset="GND" device="">
+<attribute name="SPICEPREFIX" value="G"/>
+</part>
 <part name="GND7" library="supply1" library_urn="urn:adsk.eagle:library:371" deviceset="GND" device=""/>
 <part name="U1" library="water-lib" deviceset="ESP-32S" device=""/>
@@
 <part name="R8" library="rcl" library_urn="urn:adsk.eagle:library:334" deviceset="R-EU_" device="R0805" package3d_urn="urn:adsk.eagle:package:23553/2" value="1K5"/>
 <part name="F1" library="water-lib" deviceset="SMD0805-020-16V" device=""/>
+<part name="IC1" library="water-lib" deviceset="IPS6404L-SQ-SPN" device=""/>
+<part name="R1" library="rcl" library_urn="urn:adsk.eagle:library:334" deviceset="R-EU_" device="R0805" package3d_urn="urn:adsk.eagle:package:23553/2" value="10k"/>
+<part name="+3V1" library="supply1" library_urn="urn:adsk.eagle:library:371" deviceset="+3V3" device=""/>
+<part name="GND1" library="supply1" library_urn="urn:adsk.eagle:library:371" deviceset="GND" device=""/>
+<part name="+3V2" library="supply1" library_urn="urn:adsk.eagle:library:371" deviceset="+3V3" device=""/>
+<part name="C1" library="rcl" library_urn="urn:adsk.eagle:library:334" deviceset="C-EU" device="C0805" package3d_urn="urn:adsk.eagle:package:23617/2" value="0.1uF"/>
+<part name="GND2" library="supply1" library_urn="urn:adsk.eagle:library:371" deviceset="GND" device=""/>
 </parts>
 <sheets>
@@
 <plain>
 <frame x1="-322.58" y1="60.96" x2="-157.48" y2="190.5" columns="8" rows="5" layer="91"/>
+<frame x1="-160.02" y1="190.5" x2="-53.34" y2="254" columns="8" rows="5" layer="91"/>
 </plain>
 <instances>
@@
 <attribute name="NAME" x="-298.45" y="140.716" size="1.778" layer="95" rot="R90" align="center-left"/>
 <attribute name="VALUE" x="-295.91" y="131.064" size="1.778" layer="96" rot="R90" align="center-left"/>
+</instance>
+<instance part="IC1" gate="G$1" x="-129.54" y="220.98" smashed="yes">
+<attribute name="NAME" x="-124.714" y="224.79" size="1.778" layer="95" align="center-left"/>
+<attribute name="VALUE" x="-115.316" y="225.044" size="1.778" layer="96" align="center-left"/>
+</instance>
+<instance part="R1" gate="G$1" x="-132.08" y="231.14" smashed="yes" rot="R90">
+<attribute name="NAME" x="-133.5786" y="229.87" size="1.778" layer="95" rot="R90"/>
+<attribute name="VALUE" x="-128.778" y="227.33" size="1.778" layer="96" rot="R90"/>
+</instance>
+<instance part="+3V1" gate="G$1" x="-132.08" y="241.3" smashed="yes">
+<attribute name="VALUE" x="-129.54" y="241.3" size="1.778" layer="96" rot="R90"/>
+</instance>
+<instance part="GND1" gate="1" x="-129.54" y="208.28" smashed="yes">
+<attribute name="VALUE" x="-132.08" y="205.74" size="1.778" layer="96"/>
+</instance>
+<instance part="+3V2" gate="G$1" x="-88.9" y="233.68" smashed="yes">
+<attribute name="VALUE" x="-86.36" y="233.68" size="1.778" layer="96" rot="R90"/>
+</instance>
+<instance part="C1" gate="G$1" x="-81.28" y="226.06" smashed="yes" rot="R90">
+<attribute name="NAME" x="-81.661" y="227.584" size="1.778" layer="95" rot="R90"/>
+<attribute name="VALUE" x="-76.581" y="227.584" size="1.778" layer="96" rot="R90"/>
+</instance>
+<instance part="GND2" gate="1" x="-71.12" y="226.06" smashed="yes" rot="R90">
+<attribute name="VALUE" x="-68.58" y="223.52" size="1.778" layer="96" rot="R90"/>
 </instance>
 </instances>
@@
 <pinref part="+3V4" gate="G$1" pin="+3V3"/>
 <wire x1="-119.38" y1="137.16" x2="-116.84" y2="137.16" width="0.1524" layer="91"/>
+</segment>
+<segment>
+<pinref part="R1" gate="G$1" pin="2"/>
+<wire x1="-132.08" y1="236.22" x2="-132.08" y2="238.76" width="0.1524" layer="91"/>
+<pinref part="+3V1" gate="G$1" pin="+3V3"/>
+</segment>
+<segment>
+<pinref part="IC1" gate="G$1" pin="VDD"/>
+<pinref part="+3V2" gate="G$1" pin="+3V3"/>
+<wire x1="-88.9" y1="220.98" x2="-88.9" y2="226.06" width="0.1524" layer="91"/>
+<pinref part="C1" gate="G$1" pin="1"/>
+<wire x1="-88.9" y1="226.06" x2="-88.9" y2="231.14" width="0.1524" layer="91"/>
+<wire x1="-83.82" y1="226.06" x2="-88.9" y2="226.06" width="0.1524" layer="91"/>
+<junction x="-88.9" y="226.06"/>
 </segment>
 </net>
@@
 <pinref part="U1" gate="G$1" pin="GND@4"/>
 <label x="17.78" y="114.3" size="1.778" layer="95"/>
+</segment>
+<segment>
+<pinref part="IC1" gate="G$1" pin="VSS"/>
+<pinref part="GND1" gate="1" pin="GND"/>
+<wire x1="-129.54" y1="213.36" x2="-129.54" y2="210.82" width="0.1524" layer="91"/>
+</segment>
+<segment>
+<pinref part="C1" gate="G$1" pin="2"/>
+<pinref part="GND2" gate="1" pin="GND"/>
+<wire x1="-76.2" y1="226.06" x2="-73.66" y2="226.06" width="0.1524" layer="91"/>
 </segment>
 </net>
@@
 </segment>
 </net>
+<net name="IO16" class="0">
+<segment>
+<pinref part="IC1" gate="G$1" pin="#CE"/>
+<pinref part="R1" gate="G$1" pin="1"/>
+<wire x1="-129.54" y1="220.98" x2="-132.08" y2="220.98" width="0.1524" layer="91"/>
+<wire x1="-132.08" y1="220.98" x2="-132.08" y2="226.06" width="0.1524" layer="91"/>
+<label x="-134.62" y="220.98" size="1.778" layer="95" rot="R180" xref="yes"/>
+<wire x1="-134.62" y1="220.98" x2="-132.08" y2="220.98" width="0.1524" layer="91"/>
+<junction x="-132.08" y="220.98"/>
+</segment>
+<segment>
+<pinref part="U1" gate="G$1" pin="IO16"/>
+<wire x1="10.16" y1="101.6" x2="12.7" y2="101.6" width="0.1524" layer="91"/>
+<label x="12.7" y="101.6" size="1.778" layer="95" xref="yes"/>
+</segment>
+</net>
+<net name="SD0" class="0">
+<segment>
+<pinref part="IC1" gate="G$1" pin="SO/SIO[1]"/>
+<wire x1="-129.54" y1="218.44" x2="-144.78" y2="218.44" width="0.1524" layer="91"/>
+<label x="-144.78" y="218.44" size="1.778" layer="95" rot="R180" xref="yes"/>
+</segment>
+<segment>
+<pinref part="U1" gate="G$1" pin="SD0"/>
+<wire x1="10.16" y1="83.82" x2="12.7" y2="83.82" width="0.1524" layer="91"/>
+<label x="12.7" y="83.82" size="1.778" layer="95" xref="yes"/>
+</segment>
+</net>
+<net name="SD3" class="0">
+<segment>
+<pinref part="IC1" gate="G$1" pin="SIO[2]"/>
+<wire x1="-129.54" y1="215.9" x2="-134.62" y2="215.9" width="0.1524" layer="91"/>
+<label x="-134.62" y="215.9" size="1.778" layer="95" rot="R180" xref="yes"/>
+</segment>
+<segment>
+<pinref part="U1" gate="G$1" pin="SD3"/>
+<wire x1="-25.4" y1="83.82" x2="-27.94" y2="83.82" width="0.1524" layer="91"/>
+<label x="-27.94" y="83.82" size="1.778" layer="95" rot="R180" xref="yes"/>
+</segment>
+</net>
+<net name="SD1" class="0">
+<segment>
+<pinref part="IC1" gate="G$1" pin="SI/SIO[0]"/>
+<wire x1="-88.9" y1="213.36" x2="-86.36" y2="213.36" width="0.1524" layer="91"/>
+<label x="-86.36" y="213.36" size="1.778" layer="95" xref="yes"/>
+</segment>
+<segment>
+<pinref part="U1" gate="G$1" pin="SD1"/>
+<wire x1="10.16" y1="86.36" x2="20.32" y2="86.36" width="0.1524" layer="91"/>
+<label x="20.32" y="86.36" size="1.778" layer="95" xref="yes"/>
+</segment>
+</net>
+<net name="SD2" class="0">
+<segment>
+<pinref part="IC1" gate="G$1" pin="SIO[3]"/>
+<wire x1="-88.9" y1="218.44" x2="-86.36" y2="218.44" width="0.1524" layer="91"/>
+<label x="-86.36" y="218.44" size="1.778" layer="95" xref="yes"/>
+</segment>
+<segment>
+<pinref part="U1" gate="G$1" pin="SD2"/>
+<wire x1="-25.4" y1="86.36" x2="-35.56" y2="86.36" width="0.1524" layer="91"/>
+<label x="-35.56" y="86.36" size="1.778" layer="95" rot="R180" xref="yes"/>
+</segment>
+</net>
+<net name="PSRAM_CLK" class="0">
+<segment>
+<pinref part="IC1" gate="G$1" pin="SCLK"/>
+<wire x1="-88.9" y1="215.9" x2="-78.74" y2="215.9" width="0.1524" layer="91"/>
+<label x="-78.74" y="215.9" size="1.778" layer="95" xref="yes"/>
+</segment>
+<segment>
+<pinref part="U1" gate="G$1" pin="IO17"/>
+<wire x1="10.16" y1="104.14" x2="20.32" y2="104.14" width="0.1524" layer="91"/>
+<label x="20.32" y="104.14" size="1.778" layer="95" xref="yes"/>
+</segment>
+</net>
