File: main-board/_autosave-main-board.kicad_pcb (KiCad board)
At the start: 2 copper layers, 101 x 101 mm, 83 parts, among them J101 TF-01A, J102 FH12-24S-0.5SH(55), J201 C10418, Q101 DMG1012T, Q102 Q_NPN_BCE, Q201 Q_NPN_BCE, Q202 Q_NPN_BCE, SW101 SW_DIP_x01, U101 SX1308, U102 DW06D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

Commit message: refactor
Parts:
- removed BT101: Battery_Holder, water-lib:Battery-Holder-SMD
- removed D101: D_Schottky, Diode_SMD:D_SMA_Handsoldering
- removed L101: 22uH, Inductor_SMD:L_Bourns-SRN6028
- removed Q101: DMG1012T, water-lib:SOT-523
- removed R101: 10k, Resistor_SMD:R_0805_2012Metric_Pad1.15x1.40mm_HandSolder
- removed U101: SX1308, Package_TO_SOT_SMD:SOT-23-6_Handsoldering
- added BT301: Battery_Holder, water-lib:Battery-Holder-SMD, F.Cu at (146.2, 90.2)
- added C301: 22uF, Capacitor_SMD:C_1206_3216Metric_Pad1.42x1.75mm_HandSolder, F.Cu at (64.5, 43.1)
- added C302: 0.1uF, Capacitor_SMD:C_0805_2012Metric_Pad1.15x1.40mm_HandSolder, F.Cu at (37.5, 43.4)
- added C303: 22uF, Capacitor_SMD:C_1206_3216Metric_Pad1.42x1.75mm_HandSolder, F.Cu at (56.1, 39.0)
- added C304: 1uF, Capacitor_SMD:C_0805_2012Metric_Pad1.15x1.40mm_HandSolder, F.Cu at (42.2, 43.4)
- added D301: D_Schottky, Diode_SMD:D_SMA_Handsoldering, F.Cu at (167.2, 122.5)
- added L301: 22uH, Inductor_SMD:L_Bourns-SRN6028, F.Cu at (165.4, 130.8)
- added Q301: DMG1012T, water-lib:SOT-523, F.Cu at (156.4, 48.4)
- added R301: 10k, Resistor_SMD:R_0805_2012Metric_Pad1.15x1.40mm_HandSolder, F.Cu at (158.5, 123.8)
- added R302: 2k2, Resistor_SMD:R_0805_2012Metric_Pad1.15x1.40mm_HandSolder, F.Cu at (53.9, 46.4)
- added R303: 100, Resistor_SMD:R_0805_2012Metric_Pad1.15x1.40mm_HandSolder, F.Cu at (58.7, 42.2)
- added R304: 10k, Resistor_SMD:R_0805_2012Metric_Pad1.15x1.40mm_HandSolder, F.Cu at (63.4, 38.9)
- added R305: 1k, Resistor_SMD:R_0805_2012Metric_Pad1.15x1.40mm_HandSolder, F.Cu at (68.2, 38.9)
- added R306: 27k, Resistor_SMD:R_0805_2012Metric_Pad1.15x1.40mm_HandSolder, F.Cu at (72.9, 38.9)
- added R307: 10k, Resistor_SMD:R_0805_2012Metric_Pad1.15x1.40mm_HandSolder, F.Cu at (77.7, 38.9)
- added U301: SX1308, Package_TO_SOT_SMD:SOT-23-6_Handsoldering, F.Cu at (159.2, 127.7)
- added U302: DW06D, Package_TO_SOT_SMD:SOT-23-6_Handsoldering, F.Cu at (152.3, 136.9)
Connections:
- net /VBAT renamed /BATTERY/VBAT
Routing:
- net Net-(D301-Pad1): track 0.00 -> 11.0 mm
- net Net-(D101-Pad1): track 11.0 -> 0.00 mm
- net /BATTERY/VBAT: track 119.7 -> 118.9 mm, vias 0 -> 1
- net GND: vias 72 -> 71
