File: main-board/camera.sch (KiCad schematic (older format))
At the start: 15 parts, among them J402 FH12-24S-0.5SH(55), U402 RT9011-CMGJ6

Commit message: ALPHA 1
Parts:
- added TP301: +2V8, TestPoint:TestPoint_Pad_D1.0mm, symbol Connector:TestPoint
- added TP302: +1V2, TestPoint:TestPoint_Pad_D1.0mm, symbol Connector:TestPoint
- renumbered C407 to C301, C408 to C302, C409 to C303, C406 to C304, C404 to C305, C405 to C306, J402 to J301, R405 to R301, R407 to R302, R408 to R303, R409 to R304, R410 to R305, R411 to R306, R406 to R307, U402 to U301
Connections:
- net +1V2: now also TP302.1
- net +2V8: now also TP301.1
Other:
- moved on the sheet: C301, C302, C303, C304, C305, C306, J301, R301, R302, R303, R304, R305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
