File: main-board/sd.sch (KiCad schematic (older format))
At the start: 9 parts, among them J401 TF-01A, U401 SN74LVC125ADBR

Commit message: ALPHA 1
Changed lines of the file:
@@
 $Descr A4 11693 8268
 encoding utf-8
-Sheet 4 4
+Sheet 4 5
 Title ""
 Date ""
@@
 AR Path="/5DA50BAF" Ref="J?"  Part="1"
 AR Path="/5DA30327/5DA50BAF" Ref="J401"  Part="1"
-F 0 "J?" H 2270 2885 50  0000 C CNN
+F 0 "J401" H 2270 2885 50  0000 C CNN
 F 1 "TF-01A" H 2270 2794 50  0000 C CNN
 F 2 "water-lib:TF-01A" H 3470 2460 50  0001 C CNN
@@
 AR Path="/5DA50BB5" Ref="#PWR?"  Part="1"
 AR Path="/5DA30327/5DA50BB5" Ref="#PWR0107"  Part="1"
-F 0 "#PWR?" H 1430 1540 50  0001 C CNN
+F 0 "#PWR0107" H 1430 1540 50  0001 C CNN
 F 1 "GND" H 1435 1617 50  0000 C CNN
 F 2 "" H 1430 1790 50  0001 C CNN
@@
 AR Path="/5DA50BC6" Ref="#PWR?"  Part="1"
 AR Path="/5DA30327/5DA50BC6" Ref="#PWR0108"  Part="1"
-F 0 "#PWR?" H 3780 1910 50  0001 C CNN
+F 0 "#PWR0108" H 3780 1910 50  0001 C CNN
 F 1 "+3V3" H 3795 2233 50  0000 C CNN
 F 2 "" H 3780 2060 50  0001 C CNN
@@
 AR Path="/5DA50BCD" Ref="C?"  Part="1"
 AR Path="/5DA30327/5DA50BCD" Ref="C401"  Part="1"
-F 0 "C?" H 3940 2150 50  0000 L CNN
+F 0 "C401" H 3940 2150 50  0000 L CNN
 F 1 "10uF" H 3840 1980 50  0000 L CNN
 F 2 "Capacitor_SMD:C_0805_2012Metric_Pad1.15x1.40mm_HandSolder" H 4108 1910 50  0001 C CNN
@@
 AR Path="/5DA50BD4" Ref="C?"  Part="1"
 AR Path="/5DA30327/5DA50BD4" Ref="C402"  Part="1"
-F 0 "C?" H 3940 2380 50  0000 L CNN
+F 0 "C402" H 3940 2380 50  0000 L CNN
 F 1 "0.1uF" H 3840 2210 50  0000 L CNN
 F 2 "Capacitor_SMD:C_0805_2012Metric_Pad1.15x1.40mm_HandSolder" H 4108 2140 50  0001 C CNN
@@
 AR Path="/5DA50BDA" Ref="#PWR?"  Part="1"
 AR Path="/5DA30327/5DA50BDA" Ref="#PWR0109"  Part="1"
-F 0 "#PWR?" H 4220 1910 50  0001 C CNN
+F 0 "#PWR0109" H 4220 1910 50  0001 C CNN
 F 1 "GND" H 4225 1987 50  0000 C CNN
 F 2 "" H 4220 2160 50  0001 C CNN
@@
 AR Path="/5DA50BEB" Ref="#PWR?"  Part="1"
 AR Path="/5DA30327/5DA50BEB" Ref="#PWR0110"  Part="1"
-F 0 "#PWR?" H 3450 1610 50  0001 C CNN
+F 0 "#PWR0110" H 3450 1610 50  0001 C CNN
 F 1 "GND" H 3455 1687 50  0000 C CNN
 F 2 "" H 3450 1860 50  0001 C CNN
@@
 AR Path="/5DA50BF4" Ref="R?"  Part="1"
 AR Path="/5DA30327/5DA50BF4" Ref="R401"  Part="1"
-F 0 "R?" V 3900 1760 50  0000 C CNN
+F 0 "R401" V 3900 1760 50  0000 C CNN
 F 1 "3k3" V 3820 1760 50  0000 C CNN
 F 2 "Resistor_SMD:R_0805_2012Metric_Pad1.15x1.40mm_HandSolder" H 3820 1760 50  0001 C CNN
@@
 AR Path="/5DA50BFE" Ref="#PWR?"  Part="1"
 AR Path="/5DA30327/5DA50BFE" Ref="#PWR0111"  Part="1"
-F 0 "#PWR?" H 3220 2460 50  0001 C CNN
+F 0 "#PWR0111" H 3220 2460 50  0001 C CNN
 F 1 "GND" H 3225 2537 50  0000 C CNN
 F 2 "" H 3220 2710 50  0001 C CNN
@@
 AR Path="/5DA9C676" Ref="U?"  Part="1"
 AR Path="/5DA30327/5DA9C676" Ref="U401"  Part="1"
-F 0 "U?" H 7030 2941 50  0000 C CNN
+F 0 "U401" H 7030 2941 50  0000 C CNN
 F 1 "SN74LVC125ADBR" H 7030 2850 50  0000 C CNN
 F 2 "Package_SO:TSSOP-14_4.4x5mm_P0.65mm" H 7980 1610 50  0001 C CNN
@@
 AR Path="/5DA9C682" Ref="#PWR?"  Part="1"
 AR Path="/5DA30327/5DA9C682" Ref="#PWR0112"  Part="1"
-F 0 "#PWR?" H 7030 2410 50  0001 C CNN
+F 0 "#PWR0112" H 7030 2410 50  0001 C CNN
 F 1 "GND" H 7035 2487 50  0000 C CNN
 F 2 "" H 7030 2660 50  0001 C CNN
@@
 AR Path="/5DA9C698" Ref="#PWR?"  Part="1"
 AR Path="/5DA30327/5DA9C698" Ref="#PWR0113"  Part="1"
-F 0 "#PWR?" H 7440 1410 50  0001 C CNN
+F 0 "#PWR0113" H 7440 1410 50  0001 C CNN
 F 1 "+3V3" H 7455 1733 50  0000 C CNN
 F 2 "" H 7440 1560 50  0001 C CNN
@@
 AR Path="/5DA9C69F" Ref="C?"  Part="1"
 AR Path="/5DA30327/5DA9C69F" Ref="C403"  Part="1"
-F 0 "C?" H 7580 1650 50  0000 L CNN
+F 0 "C403" H 7580 1650 50  0000 L CNN
 F 1 "0.1uF" H 7480 1480 50  0000 L CNN
 F 2 "Capacitor_SMD:C_0805_2012Metric_Pad1.15x1.40mm_HandSolder" H 7748 1410 50  0001 C CNN
@@
 AR Path="/5DA9C6AD" Ref="R?"  Part="1"
 AR Path="/5DA30327/5DA9C6AD" Ref="R402"  Part="1"
-F 0 "R?" V 6000 1960 50  0000 C CNN
+F 0 "R402" V 6000 1960 50  0000 C CNN
 F 1 "3k3" V 5920 1960 50  0000 C CNN
 F 2 "Resistor_SMD:R_0805_2012Metric_Pad1.15x1.40mm_HandSolder" H 5920 1960 50  0001 C CNN
@@
 AR Path="/5DA9C6B6" Ref="R?"  Part="1"
 AR Path="/5DA30327/5DA9C6B6" Ref="R403"  Part="1"
-F 0 "R?" V 6010 2260 50  0000 C CNN
+F 0 "R403" V 6010 2260 50  0000 C CNN
 F 1 "3k3" V 5930 2260 50  0000 C CNN
 F 2 "Resistor_SMD:R_0805_2012Metric_Pad1.15x1.40mm_HandSolder" H 5930 2260 50  0001 C CNN
@@
 AR Path="/5DA9C6BF" Ref="R?"  Part="1"
 AR Path="/5DA30327/5DA9C6BF" Ref="R404"  Part="1"
-F 0 "R?" V 8280 2260 50  0000 C CNN
+F 0 "R404" V 8280 2260 50  0000 C CNN
 F 1 "3k3" V 8200 2260 50  0000 C CNN
 F 2 "Resistor_SMD:R_0805_2012Metric_Pad1.15x1.40mm_HandSolder" H 8200 2260 50  0001 C CNN

Commit message: ALPHA 1
Parts:
- renumbered C401 to C501, C402 to C502, C403 to C503, J401 to J501, R401 to R501, R402 to R502, R403 to R503, R404 to R504, U401 to U501
Other:
- moved on the sheet: C501, C502, C503, J501, R501, R502, R503, R504, U501
