File: main-board/main-board.sch (KiCad schematic (older format))
At the start: 72 parts, among them J1 C10418, J2 FH12-24S-0.5SH(55), J3 TF-01A, Q1 Q_NPN_BCE, Q2 Q_NPN_BCE, Q3 Q_NPN_BCE, Q4 DMG1012T, SW1 SW_DIP_x01, U1 ESP-32s, U2 HT7333-A, U3 CH340E, U4 DW06D, U5 IPS6404L-SQ-SPN, U6 SX1308, U7 RT9011-CMGJ6, U8 SN74LVC125ADBR

Commit message: Mounting holes and test points
Parts:
- added H1, H2, H3, H4: MountingHole, MountingHole:MountingHole_3.2mm_M3_Pad_Via, symbol Mechanical:MountingHole
- added TP1: +2V8, TestPoint:TestPoint_Pad_D1.0mm, symbol Connector:TestPoint
- added TP2: VBAT, TestPoint:TestPoint_Pad_D1.0mm, symbol Connector:TestPoint
- added TP3: GND, TestPoint:TestPoint_Pad_D1.0mm, symbol Connector:TestPoint
- added TP4: +5V, TestPoint:TestPoint_Pad_D1.0mm, symbol Connector:TestPoint
- added TP5: +3.3V, TestPoint:TestPoint_Pad_D1.0mm, symbol Connector:TestPoint
- added TP6: +3V3, TestPoint:TestPoint_Pad_D1.0mm, symbol Connector:TestPoint
- added TP7: +1V2, TestPoint:TestPoint_Pad_D1.0mm, symbol Connector:TestPoint
Connections:
- wire segments 272 -> 279
Changed lines of the file:
@@
 	0    -1   -1   0
 $EndComp
+$Comp
+L Mechanical:MountingHole H4
+U 1 1 5D9F8791
+P 6280 6350
+F 0 "H4" H 6380 6396 50  0000 L CNN
+F 1 "MountingHole" H 6380 6305 50  0000 L CNN
+F 2 "MountingHole:MountingHole_3.2mm_M3_Pad_Via" H 6280 6350 50  0001 C CNN
+F 3 "~" H 6280 6350 50  0001 C CNN
+	1    6280 6350
+	1    0    0    -1
+$EndComp
+$Comp
+L Mechanical:MountingHole H1
+U 1 1 5DA135E4
+P 6270 6600
+F 0 "H1" H 6370 6646 50  0000 L CNN
+F 1 "MountingHole" H 6370 6555 50  0000 L CNN
+F 2 "MountingHole:MountingHole_3.2mm_M3_Pad_Via" H 6270 6600 50  0001 C CNN
+F 3 "~" H 6270 6600 50  0001 C CNN
+	1    6270 6600
+	1    0    0    -1
+$EndComp
+$Comp
+L Mechanical:MountingHole H2
+U 1 1 5DA1392B
+P 6270 6840
+F 0 "H2" H 6370 6886 50  0000 L CNN
+F 1 "MountingHole" H 6370 6795 50  0000 L CNN
+F 2 "MountingHole:MountingHole_3.2mm_M3_Pad_Via" H 6270 6840 50  0001 C CNN
+F 3 "~" H 6270 6840 50  0001 C CNN
+	1    6270 6840
+	1    0    0    -1
+$EndComp
+$Comp
+L Mechanical:MountingHole H3
+U 1 1 5DA13B73
+P 6270 7080
+F 0 "H3" H 6370 7126 50  0000 L CNN
+F 1 "MountingHole" H 6370 7035 50  0000 L CNN
+F 2 "MountingHole:MountingHole_3.2mm_M3_Pad_Via" H 6270 7080 50  0001 C CNN
+F 3 "~" H 6270 7080 50  0001 C CNN
+	1    6270 7080
+	1    0    0    -1
+$EndComp
+$Comp
+L Connector:TestPoint TP3
+U 1 1 5DA2FB24
+P 710 5880
+F 0 "TP3" V 780 6050 50  0000 R CNN
+F 1 "GND" V 620 6050 50  0000 R CNN
+F 2 "TestPoint:TestPoint_Pad_D1.0mm" H 910 5880 50  0001 C CNN
+F 3 "~" H 910 5880 50  0001 C CNN
+	1    710  5880
+	0    -1   -1   0
+$EndComp
+$Comp
+L Connector:TestPoint TP4
+U 1 1 5DA9028F
+P 710 6160
+F 0 "TP4" V 780 6330 50  0000 R CNN
+F 1 "+5V" V 620 6330 50  0000 R CNN
+F 2 "TestPoint:TestPoint_Pad_D1.0mm" H 910 6160 50  0001 C CNN
+F 3 "~" H 910 6160 50  0001 C CNN
+	1    710  6160
+	0    -1   -1   0
+$EndComp
+$Comp
+L Connector:TestPoint TP5
+U 1 1 5DA90A60
+P 710 6430
+F 0 "TP5" V 780 6600 50  0000 R CNN
+F 1 "+3.3V" V 620 6600 50  0000 R CNN
+F 2 "TestPoint:TestPoint_Pad_D1.0mm" H 910 6430 50  0001 C CNN
+F 3 "~" H 910 6430 50  0001 C CNN
+	1    710  6430
+	0    -1   -1   0
+$EndComp
+$Comp
+L Connector:TestPoint TP6
+U 1 1 5DA90FD1
+P 710 6690
+F 0 "TP6" V 780 6860 50  0000 R CNN
+F 1 "+3V3" V 620 6860 50  0000 R CNN
+F 2 "TestPoint:TestPoint_Pad_D1.0mm" H 910 6690 50  0001 C CNN
+F 3 "~" H 910 6690 50  0001 C CNN
+	1    710  6690
+	0    -1   -1   0
+$EndComp
+$Comp
+L Connector:TestPoint TP7
+U 1 1 5DA913A0
+P 710 6980
+F 0 "TP7" V 780 7150 50  0000 R CNN
+F 1 "+1V2" V 620 7150 50  0000 R CNN
+F 2 "TestPoint:TestPoint_Pad_D1.0mm" H 910 6980 50  0001 C CNN
+F 3 "~" H 910 6980 50  0001 C CNN
+	1    710  6980
+	0    -1   -1   0
+$EndComp
+$Comp
+L power:GND #PWR056
+U 1 1 5DA91749
+P 760 5880
+F 0 "#PWR056" H 760 5630 50  0001 C CNN
+F 1 "GND" H 765 5707 50  0000 C CNN
+F 2 "" H 760 5880 50  0001 C CNN
+F 3 "" H 760 5880 50  0001 C CNN
+	1    760  5880
+	0    -1   -1   0
+$EndComp
+$Comp
+L power:+5V #PWR057
+U 1 1 5DA92174
+P 760 6160
+F 0 "#PWR057" H 760 6010 50  0001 C CNN
+F 1 "+5V" H 775 6333 50  0000 C CNN
+F 2 "" H 760 6160 50  0001 C CNN
+F 3 "" H 760 6160 50  0001 C CNN
+	1    760  6160
+	0    1    1    0
+$EndComp
+$Comp
+L power:VCC #PWR058
+U 1 1 5DA9346E
+P 780 6430
+F 0 "#PWR058" H 780 6280 50  0001 C CNN
+F 1 "VCC" H 797 6603 50  0000 C CNN
+F 2 "" H 780 6430 50  0001 C CNN
+F 3 "" H 780 6430 50  0001 C CNN
+	1    780  6430
+	0    1    1    0
+$EndComp
+$Comp
+L power:+3V3 #PWR059
+U 1 1 5DA94330
+P 790 6690
+F 0 "#PWR059" H 790 6540 50  0001 C CNN
+F 1 "+3V3" H 805 6863 50  0000 C CNN
+F 2 "" H 790 6690 50  0001 C CNN
+F 3 "" H 790 6690 50  0001 C CNN
+	1    790  6690
+	0    1    1    0
+$EndComp
+$Comp
+L power:+1V2 #PWR060
+U 1 1 5DA9596A
+P 810 6980
+F 0 "#PWR060" H 810 6830 50  0001 C CNN
+F 1 "+1V2" H 825 7153 50  0000 C CNN
+F 2 "" H 810 6980 50  0001 C CNN
+F 3 "" H 810 6980 50  0001 C CNN
+	1    810  6980
+	0    1    1    0
+$EndComp
+$Comp
+L Connector:TestPoint TP1
+U 1 1 5DA972FE
+P 700 7250
+F 0 "TP1" V 770 7420 50  0000 R CNN
+F 1 "+2V8" V 610 7420 50  0000 R CNN
+F 2 "TestPoint:TestPoint_Pad_D1.0mm" H 900 7250 50  0001 C CNN
+F 3 "~" H 900 7250 50  0001 C CNN
+	1    700  7250
+	0    -1   -1   0
+$EndComp
+$Comp
+L power:+2V8 #PWR061
+U 1 1 5DA979D8
+P 810 7250
+F 0 "#PWR061" H 810 7100 50  0001 C CNN
+F 1 "+2V8" H 825 7423 50  0000 C CNN
+F 2 "" H 810 7250 50  0001 C CNN
+F 3 "" H 810 7250 50  0001 C CNN
+	1    810  7250
+	0    1    1    0
+$EndComp
+Wire Wire Line
+	710  5880 760  5880
+Wire Wire Line
+	710  6160 760  6160
+Wire Wire Line
+	710  6430 780  6430
+Wire Wire Line
+	710  6690 790  6690
+Wire Wire Line
+	710  6980 810  6980
+Wire Wire Line
+	700  7250 810  7250
+$Comp
+L Connector:TestPoint TP2
+U 1 1 5DB4294C
+P 700 7510
+F 0 "TP2" V 770 7680 50  0000 R CNN
+F 1 "VBAT" V 610 7680 50  0000 R CNN
+F 2 "TestPoint:TestPoint_Pad_D1.0mm" H 900 7510 50  0001 C CNN
+F 3 "~" H 900 7510 50  0001 C CNN
+	1    700  7510
+	0    -1   -1   0
+$EndComp
+Wire Wire Line
+	700  7510 900  7510
+Text Label 730  7510 0    50   ~ 0
+VBAT
 $EndSCHEMATC

Commit message: BOM parts
Parts:
- BT1: Aliexpress (none) -> https://www.aliexpress.com/wholesale?catId=0&initiative_id=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
- C1, C16, C2: LCSC (none) -> C15850
- C10, C11, C15, C19, C8, C9: LCSC (none) -> C24123
- C12: LCSC (none) -> C1794
- C13, C17, C18, C3, C4, C5: LCSC (none) -> C1790
- C6, C7: LCSC (none) -> C5674
- D1, D2, D3, D4: LCSC (none) -> C94691
- J1: LCSC (none) -> C10418
- L1: footprint Inductor_SMD:L_6.3x6.3_H3 -> Inductor_SMD:L_7.3x7.3_H3.5; LCSC (none) -> C237916
Changed lines of the file:
@@
 F 6 "Jing Extension of the Electronic Co." H 2550 5200 50  0001 L CNN "Manufacturer_Name"
 F 7 "C10418" H 2550 5100 50  0001 L CNN "Manufacturer_Part_Number"
+F 8 "C10418" H 1700 5700 50  0001 C CNN "LCSC"
 	1    1700 5700
 	1    0    0    -1
@@
 F 2 "Capacitor_SMD:C_0805_2012Metric_Pad1.15x1.40mm_HandSolder" H 2578 4850 50  0001 C CNN
 F 3 "~" H 2540 5000 50  0001 C CNN
+F 4 "C15850" H 2540 5000 50  0001 C CNN "LCSC"
 	1    2540 5000
 	1    0    0    -1
@@
 F 2 "Capacitor_SMD:C_0805_2012Metric_Pad1.15x1.40mm_HandSolder" H 3578 4850 50  0001 C CNN
 F 3 "~" H 3540 5000 50  0001 C CNN
+F 4 "C15850" H 3540 5000 50  0001 C CNN "LCSC"
 	1    3540 5000
 	1    0    0    -1
@@
 F 2 "LED_SMD:LED_0805_2012Metric_Pad1.15x1.40mm_HandSolder" H 1370 4950 50  0001 C CNN
 F 3 "~" H 1370 4950 50  0001 C CNN
+F 4 "C94691" H 1370 4950 50  0001 C CNN "LCSC"
 	1    1370 4950
 	1    0    0    -1
@@
 F 2 "LED_SMD:LED_0805_2012Metric_Pad1.15x1.40mm_HandSolder" H 5190 6600 50  0001 C CNN
 F 3 "~" H 5190 6600 50  0001 C CNN
+F 4 "C94691" H 5190 6600 50  0001 C CNN "LCSC"
 	1    5190 6600
 	0    -1   -1   0
@@
 F 2 "Capacitor_SMD:C_0805_2012Metric_Pad1.15x1.40mm_HandSolder" H 4228 5500 50  0001 C CNN
 F 3 "~" H 4190 5650 50  0001 C CNN
+F 4 "C1790" H 4190 5650 50  0001 C CNN "LCSC"
 	1    4190 5650
 	1    0    0    -1
@@
 F 2 "Capacitor_SMD:C_0805_2012Metric_Pad1.15x1.40mm_HandSolder" H 3678 5650 50  0001 C CNN
 F 3 "~" H 3640 5800 50  0001 C CNN
+F 4 "C1790" H 3640 5800 50  0001 C CNN "LCSC"
 	1    3640 5800
 	1    0    0    -1
@@
 F 2 "LED_SMD:LED_0805_2012Metric_Pad1.15x1.40mm_HandSolder" H 5740 7000 50  0001 C CNN
 F 3 "~" H 5740 7000 50  0001 C CNN
+F 4 "C94691" H 5740 7000 50  0001 C CNN "LCSC"
 	1    5740 7000
 	0    1    1    0
@@
 F 2 "LED_SMD:LED_0805_2012Metric_Pad1.15x1.40mm_HandSolder" H 5440 5300 50  0001 C CNN
 F 3 "~" H 5440 5300 50  0001 C CNN
+F 4 "C94691" H 5440 5300 50  0001 C CNN "LCSC"
 	1    5440 5300
 	-1   0    0    1
@@
 F 2 "water-lib:Battery-Holder-SMD" V 870 1330 50  0001 C CNN
 F 3 "~" V 1040 1330 50  0001 C CNN
+F 4 "https://www.aliexpress.com/wholesale?catId=0&initiative_id=SB_20191008062912&SearchText=battery+holder+18650+smd&switch_new_app=y" H 1040 1270 50  0001 C CNN "Aliexpress"
 	1    1040 1270
 	1    0    0    -1
@@
 F 2 "Capacitor_SMD:C_0805_2012Metric_Pad1.15x1.40mm_HandSolder" H 1538 1350 50  0001 C CNN
 F 3 "~" H 1500 1500 50  0001 C CNN
+F 4 "C1790" H 1500 1500 50  0001 C CNN "LCSC"
 	1    1500 1500
 	1    0    0    -1
@@
 F 2 "Capacitor_SMD:C_0805_2012Metric_Pad1.15x1.40mm_HandSolder" H 2828 2190 50  0001 C CNN
 F 3 "~" H 2790 2340 50  0001 C CNN
+F 4 "C5674" H 2790 2340 50  0001 C CNN "LCSC"
 	1    2790 2340
 	1    0    0    -1
@@
 F 0 "L1" V 2120 2060 50  0000 C CNN
 F 1 "22uH" V 2029 2060 50  0000 C CNN
-F 2 "Inductor_SMD:L_6.3x6.3_H3" H 1930 2060 50  0001 C CNN
+F 2 "Inductor_SMD:L_7.3x7.3_H3.5" H 1930 2060 50  0001 C CNN
 F 3 "~" H 1930 2060 50  0001 C CNN
+F 4 "C237916" H 1930 2060 50  0001 C CNN "LCSC"
 	1    1930 2060
 	0    -1   -1   0
@@
 F 2 "Capacitor_SMD:C_0805_2012Metric_Pad1.15x1.40mm_HandSolder" H 898 2460 50  0001 C CNN
 F 3 "~" H 860 2610 50  0001 C CNN
+F 4 "C5674" H 860 2610 50  0001 C CNN "LCSC"
 	1    860  2610
 	1    0    0    -1
@@
 F 2 "Capacitor_SMD:C_0805_2012Metric_Pad1.15x1.40mm_HandSolder" H 10158 1190 50  0001 C CNN
 F 3 "~" H 10120 1340 50  0001 C CNN
+F 4 "C24123" H 10120 1340 50  0001 C CNN "LCSC"
 	1    10120 1340
 	0    1    1    0
@@
 F 2 "Capacitor_SMD:C_0805_2012Metric_Pad1.15x1.40mm_HandSolder" H 10948 2590 50  0001 C CNN
 F 3 "~" H 10910 2740 50  0001 C CNN
+F 4 "C24123" H 10910 2740 50  0001 C CNN "LCSC"
 	1    10910 2740
 	0    1    1    0
@@
 F 2 "Capacitor_SMD:C_0805_2012Metric_Pad1.15x1.40mm_HandSolder" H 10318 2490 50  0001 C CNN
 F 3 "~" H 10280 2640 50  0001 C CNN
+F 4 "C24123" H 10280 2640 50  0001 C CNN "LCSC"
 	1    10280 2640
 	0    1    1    0
@@
 F 2 "Capacitor_SMD:C_0805_2012Metric_Pad1.15x1.40mm_HandSolder" H 9158 2490 50  0001 C CNN
 F 3 "~" H 9120 2640 50  0001 C CNN
+F 4 "C24123" H 9120 2640 50  0001 C CNN "LCSC"
 	1    9120 2640
 	0    1    1    0
@@
 F 2 "Capacitor_SMD:C_0805_2012Metric_Pad1.15x1.40mm_HandSolder" H 10538 5070 50  0001 C CNN
 F 3 "~" H 10500 5220 50  0001 C CNN
+F 4 "C1794" H 10500 5220 50  0001 C CNN "LCSC"
 	1    10500 5220
 	0    1    1    0
@@
 F 2 "Capacitor_SMD:C_0805_2012Metric_Pad1.15x1.40mm_HandSolder" H 10988 5370 50  0001 C CNN
 F 3 "~" H 10950 5520 50  0001 C CNN
+F 4 "C1790" H 10950 5520 50  0001 C CNN "LCSC"
 	1    10950 5520
 	0    1    1    0
@@
 F 2 "Capacitor_SMD:C_0805_2012Metric_Pad1.15x1.40mm_HandSolder" H 9928 3890 50  0001 C CNN
 F 3 "~" H 9890 4040 50  0001 C CNN
+F 4 "C24123" H 9890 4040 50  0001 C CNN "LCSC"
 	1    9890 4040
 	-1   0    0    1
@@
 F 2 "Capacitor_SMD:C_0805_2012Metric_Pad1.15x1.40mm_HandSolder" H 4008 3420 50  0001 C CNN
 F 3 "~" H 3970 3570 50  0001 C CNN
+F 4 "C15850" H 3970 3570 50  0001 C CNN "LCSC"
 	1    3970 3570
 	0    1    1    0
@@
 F 2 "Capacitor_SMD:C_0805_2012Metric_Pad1.15x1.40mm_HandSolder" H 4008 3650 50  0001 C CNN
 F 3 "~" H 3970 3800 50  0001 C CNN
+F 4 "C1790" H 3970 3800 50  0001 C CNN "LCSC"
 	1    3970 3800
 	0    1    1    0
@@
 F 2 "Capacitor_SMD:C_0805_2012Metric_Pad1.15x1.40mm_HandSolder" H 6688 3330 50  0001 C CNN
 F 3 "~" H 6650 3480 50  0001 C CNN
+F 4 "C1790" H 6650 3480 50  0001 C CNN "LCSC"
 	1    6650 3480
 	0    1    1    0
@@
 F 2 "Capacitor_SMD:C_0805_2012Metric_Pad1.15x1.40mm_HandSolder" H 8098 2390 50  0001 C CNN
 F 3 "~" H 8060 2540 50  0001 C CNN
+F 4 "C24123" H 8060 2540 50  0001 C CNN "LCSC"
 	1    8060 2540
 	-1   0    0    1

Commit message: BOM parts 2
Parts:
- C6, C7: footprint Capacitor_SMD:C_0805_2012Metric_Pad1.15x1.40mm_HandSolder -> Capacitor_SMD:C_1206_3216Metric_Pad1.42x1.75mm_HandSolder; LCSC C5674 -> C87996
- D5: footprint Diode_SMD:D_0805_2012Metric_Pad1.15x1.40mm_HandSolder -> Diode_SMD:D_SMA_Handsoldering; LCSC (none) -> C274651
- L1: footprint Inductor_SMD:L_7.3x7.3_H3.5 -> Inductor_SMD:L_Bourns-SRN6028; LCSC C237916 -> C266430
- R1, R13, R2, R25, R26, R6: LCSC (none) -> C79496
- R10, R11, R12, R16, R18, R19, R20, R28, R7, R9: LCSC (none) -> C180849
- R14, R15, R17: LCSC (none) -> C336873
- R21, R22, R23, R24: LCSC (none) -> C160077
- R27: LCSC (none) -> C317283
- R3, R4: LCSC (none) -> C336856
- R5: LCSC (none) -> C230647
- R8: LCSC (none) -> C203855
- SW1: footprint Button_Switch_SMD:SW_SPST_CK_RS282G05A3 -> Button_Switch_SMD:SW_SPST_B3U-1000P; LCSC (none) -> C231329
Changed lines of the file:
@@
 F 2 "Resistor_SMD:R_0805_2012Metric_Pad1.15x1.40mm_HandSolder" H 880 4950 50  0001 C CNN
 F 3 "~" H 880 4950 50  0001 C CNN
+F 4 "C79496" H 880 4950 50  0001 C CNN "LCSC"
 	1    880  4950
 	0    1    1    0
@@
 F 2 "Resistor_SMD:R_0805_2012Metric_Pad1.15x1.40mm_HandSolder" H 5190 7050 50  0001 C CNN
 F 3 "~" H 5190 7050 50  0001 C CNN
+F 4 "C79496" H 5190 7050 50  0001 C CNN "LCSC"
 	1    5190 7050
 	-1   0    0    1
@@
 F 2 "Resistor_SMD:R_0805_2012Metric_Pad1.15x1.40mm_HandSolder" H 5740 5550 50  0001 C CNN
 F 3 "~" H 5740 5550 50  0001 C CNN
+F 4 "C336856" H 5740 5550 50  0001 C CNN "LCSC"
 	1    5740 5550
 	-1   0    0    1
@@
 F 2 "Resistor_SMD:R_0805_2012Metric_Pad1.15x1.40mm_HandSolder" H 5740 6500 50  0001 C CNN
 F 3 "~" H 5740 6500 50  0001 C CNN
+F 4 "C336856" H 5740 6500 50  0001 C CNN "LCSC"
 	1    5740 6500
 	-1   0    0    1
@@
 F 2 "Resistor_SMD:R_0805_2012Metric_Pad1.15x1.40mm_HandSolder" H 1500 930 50  0001 C CNN
 F 3 "~" H 1500 930 50  0001 C CNN
+F 4 "C230647" H 1500 930 50  0001 C CNN "LCSC"
 	1    1500 930
 	-1   0    0    1
@@
 F 2 "Resistor_SMD:R_0805_2012Metric_Pad1.15x1.40mm_HandSolder" H 2770 1390 50  0001 C CNN
 F 3 "~" H 2770 1390 50  0001 C CNN
+F 4 "C79496" H 2770 1390 50  0001 C CNN "LCSC"
 	1    2770 1390
 	-1   0    0    1
@@
 F 2 "Resistor_SMD:R_0805_2012Metric_Pad1.15x1.40mm_HandSolder" H 2540 2630 50  0001 C CNN
 F 3 "~" H 2540 2630 50  0001 C CNN
+F 4 "C180849" H 2540 2630 50  0001 C CNN "LCSC"
 	1    2540 2630
 	0    -1   -1   0
@@
 F 0 "C7" H 2660 2430 50  0000 L CNN
 F 1 "22uF" H 2560 2260 50  0000 L CNN
-F 2 "Capacitor_SMD:C_0805_2012Metric_Pad1.15x1.40mm_HandSolder" H 2828 2190 50  0001 C CNN
-F 3 "~" H 2790 2340 50  0001 C CNN
-F 4 "C5674" H 2790 2340 50  0001 C CNN "LCSC"
+F 2 "Capacitor_SMD:C_1206_3216Metric_Pad1.42x1.75mm_HandSolder" H 2828 2190 50  0001 C CNN
+F 3 "https://datasheet.lcsc.com/szlcsc/Samsung-Electro-Mechanics-CL31B226KPHNNNE_C87996.pdf" H 2790 2340 50  0001 C CNN
+F 4 "C87996" H 2790 2340 50  0001 C CNN "LCSC"
 	1    2790 2340
 	1    0    0    -1
@@
 F 0 "L1" V 2120 2060 50  0000 C CNN
 F 1 "22uH" V 2029 2060 50  0000 C CNN
-F 2 "Inductor_SMD:L_7.3x7.3_H3.5" H 1930 2060 50  0001 C CNN
-F 3 "~" H 1930 2060 50  0001 C CNN
-F 4 "C237916" H 1930 2060 50  0001 C CNN "LCSC"
+F 2 "Inductor_SMD:L_Bourns-SRN6028" H 1930 2060 50  0001 C CNN
+F 3 "https://datasheet.lcsc.com/szlcsc/ShunXiang-Connaught-Elec-SMNR6028-220MT_C266430.pdf" H 1930 2060 50  0001 C CNN
+F 4 "C266430" H 1930 2060 50  0001 C CNN "LCSC"
 	1    1930 2060
 	0    -1   -1   0
@@
 F 2 "Resistor_SMD:R_0805_2012Metric_Pad1.15x1.40mm_HandSolder" H 1180 2310 50  0001 C CNN
 F 3 "~" H 1180 2310 50  0001 C CNN
+F 4 "C180849" H 1180 2310 50  0001 C CNN "LCSC"
 	1    1180 2310
 	1    0    0    -1
@@
 F 2 "Resistor_SMD:R_0805_2012Metric_Pad1.15x1.40mm_HandSolder" H 1180 2940 50  0001 C CNN
 F 3 "~" H 1180 2940 50  0001 C CNN
+F 4 "C203855" H 1180 2940 50  0001 C CNN "LCSC"
 	1    1180 2940
 	1    0    0    -1
@@
 F 0 "C6" H 730 2700 50  0000 L CNN
 F 1 "22uF" H 630 2530 50  0000 L CNN
-F 2 "Capacitor_SMD:C_0805_2012Metric_Pad1.15x1.40mm_HandSolder" H 898 2460 50  0001 C CNN
-F 3 "~" H 860 2610 50  0001 C CNN
-F 4 "C5674" H 860 2610 50  0001 C CNN "LCSC"
+F 2 "Capacitor_SMD:C_1206_3216Metric_Pad1.42x1.75mm_HandSolder" H 898 2460 50  0001 C CNN
+F 3 "https://datasheet.lcsc.com/szlcsc/Samsung-Electro-Mechanics-CL31B226KPHNNNE_C87996.pdf" H 860 2610 50  0001 C CNN
+F 4 "C87996" H 860 2610 50  0001 C CNN "LCSC"
 	1    860  2610
 	1    0    0    -1
@@
 F 0 "D5" H 1450 1844 50  0000 C CNN
 F 1 "D_Schottky" H 1450 1935 50  0000 C CNN
-F 2 "Diode_SMD:D_0805_2012Metric_Pad1.15x1.40mm_HandSolder" H 1450 2060 50  0001 C CNN
-F 3 "~" H 1450 2060 50  0001 C CNN
+F 2 "Diode_SMD:D_SMA_Handsoldering" H 1450 2060 50  0001 C CNN
+F 3 "https://datasheet.lcsc.com/szlcsc/ON-Semicon-ON-MBRA210ET3G_C274651.pdf" H 1450 2060 50  0001 C CNN
+F 4 "C274651" H 1450 2060 50  0001 C CNN "LCSC"
 	1    1450 2060
 	-1   0    0    1
@@
 F 2 "Resistor_SMD:R_0805_2012Metric_Pad1.15x1.40mm_HandSolder" H 8750 1260 50  0001 C CNN
 F 3 "~" H 8750 1260 50  0001 C CNN
+F 4 "C180849" H 8750 1260 50  0001 C CNN "LCSC"
 	1    8750 1260
 	1    0    0    -1
@@
 F 2 "Resistor_SMD:R_0805_2012Metric_Pad1.15x1.40mm_HandSolder" H 9150 3090 50  0001 C CNN
 F 3 "~" H 9150 3090 50  0001 C CNN
+F 4 "C180849" H 9150 3090 50  0001 C CNN "LCSC"
 	1    9150 3090
 	1    0    0    -1
@@
 F 2 "Resistor_SMD:R_0805_2012Metric_Pad1.15x1.40mm_HandSolder" H 10210 3090 50  0001 C CNN
 F 3 "~" H 10210 3090 50  0001 C CNN
+F 4 "C180849" H 10210 3090 50  0001 C CNN "LCSC"
 	1    10210 3090
 	1    0    0    -1
@@
 F 2 "Resistor_SMD:R_0805_2012Metric_Pad1.15x1.40mm_HandSolder" H 7980 5720 50  0001 C CNN
 F 3 "~" H 7980 5720 50  0001 C CNN
+F 4 "C79496" H 7980 5720 50  0001 C CNN "LCSC"
 	1    7980 5720
 	0    1    1    0
@@
 F 2 "Resistor_SMD:R_0805_2012Metric_Pad1.15x1.40mm_HandSolder" H 6400 1640 50  0001 C CNN
 F 3 "~" H 6400 1640 50  0001 C CNN
+F 4 "C180849" H 6400 1640 50  0001 C CNN "LCSC"
 	1    6400 1640
 	0    -1   -1   0
@@
 F 2 "Resistor_SMD:R_0805_2012Metric_Pad1.15x1.40mm_HandSolder" H 10260 3890 50  0001 C CNN
 F 3 "~" H 10260 3890 50  0001 C CNN
+F 4 "C336873" H 10260 3890 50  0001 C CNN "LCSC"
 	1    10260 3890
 	0    1    1    0
@@
 F 2 "Resistor_SMD:R_0805_2012Metric_Pad1.15x1.40mm_HandSolder" H 3450 2040 50  0001 C CNN
 F 3 "~" H 3450 2040 50  0001 C CNN
+F 4 "C336873" H 3450 2040 50  0001 C CNN "LCSC"
 	1    3450 2040
 	0    1    1    0
@@
 F 2 "Resistor_SMD:R_0805_2012Metric_Pad1.15x1.40mm_HandSolder" H 3450 2140 50  0001 C CNN
 F 3 "~" H 3450 2140 50  0001 C CNN
+F 4 "C336873" H 3450 2140 50  0001 C CNN "LCSC"
 	1    3450 2140
 	0    1    1    0
@@
 F 0 "SW1" H 6760 5397 50  0000 C CNN
 F 1 "SW_DIP_x01" H 6760 5306 50  0000 C CNN
-F 2 "Button_Switch_SMD:SW_SPST_CK_RS282G05A3" H 6760 5130 50  0001 C CNN
+F 2 "Button_Switch_SMD:SW_SPST_B3U-1000P" H 6760 5130 50  0001 C CNN
 F 3 "~" H 6760 5130 50  0001 C CNN
+F 4 "C231329" H 6760 5130 50  0001 C CNN "LCSC"
 	1    6760 5130
 	1    0    0    -1
@@
 F 2 "Resistor_SMD:R_0805_2012Metric_Pad1.15x1.40mm_HandSolder" H 7290 4880 50  0001 C CNN
 F 3 "~" H 7290 4880 50  0001 C CNN
+F 4 "C180849" H 7290 4880 50  0001 C CNN "LCSC"
 	1    7290 4880
 	1    0    0    -1
@@
 F 2 "Resistor_SMD:R_0805_2012Metric_Pad1.15x1.40mm_HandSolder" H 2200 7440 50  0001 C CNN
 F 3 "~" H 2200 7440 50  0001 C CNN
+F 4 "C180849" H 2200 7440 50  0001 C CNN "LCSC"
 	1    2200 7440
 	0    1    1    0
@@
 F 2 "Resistor_SMD:R_0805_2012Metric_Pad1.15x1.40mm_HandSolder" H 2200 6850 50  0001 C CNN
 F 3 "~" H 2200 6850 50  0001 C CNN
+F 4 "C180849" H 2200 6850 50  0001 C CNN "LCSC"
 	1    2200 6850
 	0    1    1    0
@@
 F 2 "Resistor_SMD:R_0805_2012Metric_Pad1.15x1.40mm_HandSolder" H 3720 3270 50  0001 C CNN
 F 3 "~" H 3720 3270 50  0001 C CNN
+F 4 "C160077" H 3720 3270 50  0001 C CNN "LCSC"
 	1    3720 3270
 	0    -1   -1   0
@@
 F 2 "Resistor_SMD:R_0805_2012Metric_Pad1.15x1.40mm_HandSolder" H 4860 3880 50  0001 C CNN
 F 3 "~" H 4860 3880 50  0001 C CNN
+F 4 "C160077" H 4860 3880 50  0001 C CNN "LCSC"
 	1    4860 3880
 	0    -1   -1   0
@@
 F 2 "Resistor_SMD:R_0805_2012Metric_Pad1.15x1.40mm_HandSolder" H 4870 4180 50  0001 C CNN
 F 3 "~" H 4870 4180 50  0001 C CNN
+F 4 "C160077" H 4870 4180 50  0001 C CNN "LCSC"
 	1    4870 4180
 	0    -1   -1   0
@@
 F 2 "Resistor_SMD:R_0805_2012Metric_Pad1.15x1.40mm_HandSolder" H 7140 4180 50  0001 C CNN
 F 3 "~" H 7140 4180 50  0001 C CNN
+F 4 "C160077" H 7140 4180 50  0001 C CNN "LCSC"
 	1    7140 4180
 	0    -1   -1   0
@@
 F 2 "Resistor_SMD:R_0805_2012Metric_Pad1.15x1.40mm_HandSolder" H 7810 3760 50  0001 C CNN
 F 3 "~" H 7810 3760 50  0001 C CNN
+F 4 "C79496" H 7810 3760 50  0001 C CNN "LCSC"
 	1    7810 3760
 	0    -1   -1   0
@@
 F 2 "Resistor_SMD:R_0805_2012Metric_Pad1.15x1.40mm_HandSolder" H 8410 4280 50  0001 C CNN
 F 3 "~" H 8410 4280 50  0001 C CNN
+F 4 "C79496" H 8410 4280 50  0001 C CNN "LCSC"
 	1    8410 4280
 	-1   0    0    1
@@
 F 2 "Resistor_SMD:R_0805_2012Metric_Pad1.15x1.40mm_HandSolder" H 7770 1560 50  0001 C CNN
 F 3 "~" H 7770 1560 50  0001 C CNN
+F 4 "C317283" H 7770 1560 50  0001 C CNN "LCSC"
 	1    7770 1560
 	1    0    0    -1
@@
 F 2 "Resistor_SMD:R_0805_2012Metric_Pad1.15x1.40mm_HandSolder" H 7770 2530 50  0001 C CNN
 F 3 "~" H 7770 2530 50  0001 C CNN
+F 4 "C180849" H 7770 2530 50  0001 C CNN "LCSC"
 	1    7770 2530
 	1    0    0    -1
