File: battery-charging/battery-charging.kicad_pcb (KiCad board)
At the start: 2 copper layers, 38 x 16.8 mm, 20 parts, among them J101 USB_B_Micro, J102 BAT-, J103 BAT+, U101 TC4056A, U102 MT3608

Commit message: Smaller battery holder
Routing:
- net GND: track 2.92 -> 5.51 mm, vias 10 -> 14
- net +5V: track 42.1 -> 43.4 mm
Changed lines of the file:
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@@
-(kicad_pcb (version 20171130) (host pcbnew "(5.1.4)-1")
+(kicad_pcb (version 20171130) (host pcbnew "(5.1.4-0-10_14)")
   (general
     (thickness 1.6)
     (drawings 4)
-    (tracks 95)
+    (tracks 102)
     (zones 0)
     (modules 20)
@@
   (via (at 56.85 120.5) (size 0.8) (drill 0.4) (layers F.Cu B.Cu) (net 1))
   (via (at 67.9 125.5) (size 0.8) (drill 0.4) (layers F.Cu B.Cu) (net 1))
+  (via (at 58.4 115.8) (size 0.8) (drill 0.4) (layers F.Cu B.Cu) (net 1))
+  (via (at 58.2 112.75) (size 0.8) (drill 0.4) (layers F.Cu B.Cu) (net 1))
+  (segment (start 60.305 112.75) (end 60.65 113.095) (width 0.25) (layer F.Cu) (net 1))
+  (segment (start 58.2 112.75) (end 60.305 112.75) (width 0.25) (layer F.Cu) (net 1))
+  (via (at 71.65 113.15) (size 0.8) (drill 0.4) (layers F.Cu B.Cu) (net 1))
+  (via (at 56.45 124.45) (size 0.8) (drill 0.4) (layers F.Cu B.Cu) (net 1))
   (segment (start 53.873372 118.076628) (end 53.25 118.7) (width 0.25) (layer F.Cu) (net 2))
   (segment (start 54.27501 117.67499) (end 53.873372 118.076628) (width 0.25) (layer F.Cu) (net 2))
@@
   (segment (start 60.65 116.905) (end 60.65 123.25) (width 0.25) (layer F.Cu) (net 2))
   (segment (start 63.7 124.3) (end 61.7 124.3) (width 0.25) (layer F.Cu) (net 2))
-  (segment (start 68.52929 112.67429) (end 68.95 113.095) (width 0.25) (layer F.Cu) (net 2))
-  (segment (start 58.34182 112.41999) (end 68.27499 112.41999) (width 0.25) (layer F.Cu) (net 2))
-  (segment (start 57.24999 113.51182) (end 58.34182 112.41999) (width 0.25) (layer F.Cu) (net 2))
-  (segment (start 57.24999 114.88818) (end 57.24999 113.51182) (width 0.25) (layer F.Cu) (net 2))
-  (segment (start 68.27499 112.41999) (end 68.52929 112.67429) (width 0.25) (layer F.Cu) (net 2))
-  (segment (start 58.67182 116.31001) (end 57.24999 114.88818) (width 0.25) (layer F.Cu) (net 2))
-  (segment (start 60.05501 116.31001) (end 58.67182 116.31001) (width 0.25) (layer F.Cu) (net 2))
-  (segment (start 60.65 116.905) (end 60.05501 116.31001) (width 0.25) (layer F.Cu) (net 2))
   (segment (start 65.12 123.25) (end 66.15 123.25) (width 0.25) (layer F.Cu) (net 2))
   (segment (start 64.693372 123.676628) (end 65.12 123.25) (width 0.25) (layer F.Cu) (net 2))
   (segment (start 64.323372 123.676628) (end 64.693372 123.676628) (width 0.25) (layer F.Cu) (net 2))
   (segment (start 63.7 124.3) (end 64.323372 123.676628) (width 0.25) (layer F.Cu) (net 2))
+  (segment (start 68.52929 112.67429) (end 68.95 113.095) (width 0.25) (layer F.Cu) (net 2))
+  (segment (start 68.005 112.15) (end 68.52929 112.67429) (width 0.25) (layer F.Cu) (net 2))
+  (segment (start 57.65 112.15) (end 68.005 112.15) (width 0.25) (layer F.Cu) (net 2))
+  (segment (start 57.24999 112.55001) (end 57.65 112.15) (width 0.25) (layer F.Cu) (net 2))
+  (segment (start 60.645 116.9) (end 58.25 116.9) (width 0.25) (layer F.Cu) (net 2))
+  (segment (start 57.24999 115.89999) (end 57.24999 112.55001) (width 0.25) (layer F.Cu) (net 2))
+  (segment (start 58.25 116.9) (end 57.24999 115.89999) (width 0.25) (layer F.Cu) (net 2))
+  (segment (start 60.65 116.905) (end 60.645 116.9) (width 0.25) (layer F.Cu) (net 2))
   (segment (start 78.275 113.05) (end 80 113.05) (width 0.25) (layer F.Cu) (net 3))
   (segment (start 77.4 113.925) (end 78.275 113.05) (width 0.25) (layer F.Cu) (net 3))
@@
   (segment (start 49.99 117.25) (end 52.22499 115.01501) (width 0.25) (layer F.Cu) (net 6))
   (segment (start 49.05 117.25) (end 49.99 117.25) (width 0.25) (layer F.Cu) (net 6))
+  (segment (start 73.5 111.875) (end 75.4 111.875) (width 0.25) (layer F.Cu) (net 6))
   (segment (start 72.7 111.875) (end 73.5 111.875) (width 0.25) (layer F.Cu) (net 6))
-  (segment (start 55.075 111.875) (end 72.7 111.875) (width 0.25) (layer F.Cu) (net 6))
-  (segment (start 54.05 112.9) (end 55.075 111.875) (width 0.25) (layer F.Cu) (net 6))
+  (segment (start 55.25 111.7) (end 72.525 111.7) (width 0.25) (layer F.Cu) (net 6))
+  (segment (start 54.05 112.9) (end 55.25 111.7) (width 0.25) (layer F.Cu) (net 6))
+  (segment (start 72.525 111.7) (end 72.7 111.875) (width 0.25) (layer F.Cu) (net 6))
   (segment (start 53.25 112.9) (end 54.05 112.9) (width 0.25) (layer F.Cu) (net 6))
-  (segment (start 73.5 111.875) (end 75.4 111.875) (width 0.25) (layer F.Cu) (net 6))
   (segment (start 75.4 115.9) (end 73.7 117.6) (width 0.25) (layer F.Cu) (net 7))
   (segment (start 75.4 113.925) (end 75.4 115.9) (width 0.25) (layer F.Cu) (net 7))
